File: PCB Design/asl/asl.kicad_pcb (KiCad board)
At the start: 2 copper layers, 49 x 97 mm, 12 parts, among them J1 Conn_01x02_Socket, J2 Conn_01x02_Socket, J3 Conn_01x02_Socket, J4 Conn_01x02_Socket, J5 Conn_01x02_Socket, J6 Conn_01x06_Pin

Commit message: UPLOAD PCB Files
Parts:
- added G***: LOGO, Kicad Graphics:osu, F.Cu at (146.0, 69.0)
- added G***: LOGO, Kicad Graphics:rps, F.Cu at (145.5, 108.5)
- added G***: LOGO, Kicad Graphics:10179, B.Cu at (149.5, 124.5)
- added G***: LOGO, Kicad Graphics:luffy, B.Cu at (146.0, 70.0)
- added G***: LOGO, Kicad Graphics:1222, B.Cu at (144.0, 108.0)
Routing:
- net GND: track 151.7 -> 0.00 mm
- net Net-(A1-DAC1/A1): track 147.3 -> 84.6 mm
- net Net-(A1-DAC2/A0): track 122.3 -> 76.8 mm
- net +3V3: track 182.8 -> 189.2 mm
- net Net-(A1-SDA/IO23): track 122.9 -> 126.3 mm
- net Net-(A1-I39/A3): track 74.9 -> 71.7 mm
- net Net-(A1-SCL/IO22): track 115.0 -> 117.1 mm
- net Net-(A1-IO36/A4): track 46.7 -> 44.6 mm
- net Net-(A1-I34/A2): track 83.0 -> 82.3 mm
- added copper zone on B.Cu, net GND
- added copper zone on F.Cu, net GND
Other:
- board text added: "3v3"
- board text added: "An April without you is here..."
- board text added: "ECE 5466 Team 7"
- board text added: "GND"
- board text added: "JLCJLCJLCJLC"
- board text added: "Master Chief, do you mind telling me what you're doing in Fortnite? Sir, I'm thinking MIKU MIKU OOOO WEEE OOOO"
- board text added: "Ohio Against the World"
- board text added: "SCL"
- board text added: "SDA"
